File: PDB/_autosave-PDB.kicad_sch (KiCad schematic)
At the start: 2 parts, among them U1 Anderson_Horizontal

Commit message: added pdb backups
Parts:
- Battery1: footprint (none) -> PiE_Footprints:XT60_F
Changed lines of the file:
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@@
       (effects (font (size 1.27 1.27)) (justify left))
     )
-    (property "Footprint" "" (id 2) (at 78.74 26.67 0)
+    (property "Footprint" "PiE_Footprints:XT60_F" (id 2) (at 78.74 26.67 0)
       (effects (font (size 1.27 1.27)) hide)
     )
@@
     )
     (path "/61f06b21-2f97-41e2-9bcc-b68f2e7b5723"
-      (reference "Battery1") (unit 1) (value "XT60_F") (footprint "")
+      (reference "Battery1") (unit 1) (value "XT60_F") (footprint "PiE_Footprints:XT60_F")
     )
     (path "/cc06864b-7a29-42b8-ae65-4c9e7f6eecfb"
