File: PDB/PDB.kicad_pcb (KiCad board)
At the start: 2 copper layers, 112.1 x 88.3 mm, 56 parts, among them J1 Conn_01x02, J2 Conn_01x04, Q1 s8050_JSMSEMI, SW2 SW_SPDT, Sw1 D-SWITCH_MR5-111-C5N-BB, U2 CH340G, U3 PCF8574, Y1 12MHz

Commit message: idk when this was
Other:
- board text added: "Hole diameter is 127.5mil = 3.24mm"
Changed lines of the file:
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@@
     (pad_to_mask_clearance 0)
     (pcbplotparams
-      (layerselection 0x00010fc_ffffffff)
+      (layerselection 0x00013e0_7ffffffe)
       (disableapertmacros false)
       (usegerberextensions false)
@@
       (sketchpadsonfab false)
       (subtractmaskfromsilk false)
-      (outputformat 1)
+      (outputformat 4)
       (mirror false)
       (drillshape 0)
       (scaleselection 1)
-      (outputdirectory "JLC/CPL/")
+      (outputdirectory "JLC/")
     )
   )
@@
     )
   )
+  (gr_line (start 103.7336 65.1256) (end 100.4824 65.1256) (layer "Dwgs.User") (width 0.15))
+  (gr_line (start 102.108 63.5) (end 102.108 66.7512) (layer "Dwgs.User") (width 0.15))
+  (gr_line (start 144.8308 65.1256) (end 148.082 65.1256) (layer "Dwgs.User") (width 0.15))
+  (gr_line (start 146.4564 63.5) (end 146.4564 66.7512) (layer "Dwgs.User") (width 0.15))
   (gr_rect (start 57.531 16.891) (end 169.672 105.156) (layer "Edge.Cuts") (width 0.1) (fill none))
   (gr_text "5v" (at 127.6858 51.816) (layer "B.SilkS")
@@
     (effects (font (size 1 1) (thickness 0.15)))
   )
+  (gr_text "Hole diameter is 127.5mil = 3.24mm" (at 152.7556 131.8514) (layer "Dwgs.User")
+    (effects (font (size 1 1) (thickness 0.15)))
+  )
+  (dimension (type orthogonal) (layer "Cmts.User")
+    (pts (xy 169.672 16.891) (xy 169.672 105.156))
+    (height 28.575)
+    (orientation 1)
+    (gr_text "3475.0000 mils" (at 197.097 61.0235 90) (layer "Cmts.User")
+      (effects (font (size 1 1) (thickness 0.15)))
+    )
+    (format (units 3) (units_format 1) (precision 4))
+    (style (thickness 0.15) (arrow_length 1.27) (text_position_mode 0) (extension_height 0.58642) (extension_offset 0.5) keep_text_aligned)
+  )
+  (dimension (type orthogonal) (layer "Cmts.User")
+    (pts (xy 146.4564 65.1256) (xy 152.8834 102.0064))
+    (height 37.2364)
+    (orientation 1)
+    (gr_text "1452.0000 mils" (at 182.5428 83.566 90) (layer "Cmts.User")
+      (effects (font (size 1 1) (thickness 0.15)))
+    )
+    (format (units 3) (units_format 1) (precision 4))
+    (style (thickness 0.15) (arrow_length 1.27) (text_position_mode 0) (extension_height 0.58642) (extension_offset 0.5) keep_text_aligned)
+  )
+  (dimension (type orthogonal) (layer "Cmts.User")
+    (pts (xy 102.108 65.1256) (xy 146.4564 65.1256))
+    (height 52.5272)
+    (orientation 0)
+    (gr_text "1746.0000 mils" (at 124.2822 116.5028) (layer "Cmts.User")
+      (effects (font (size 1 1) (thickness 0.15)))
+    )
+    (format (units 3) (units_format 1) (precision 4))
+    (style (thickness 0.15) (arrow_length 1.27) (text_position_mode 0) (extension_height 0.58642) (extension_offset 0.5) keep_text_aligned)
+  )
+  (dimension (type orthogonal) (layer "Cmts.User")
+    (pts (xy 57.531 105.156) (xy 169.672 105.156))
+    (height 31.2166)
+    (orientation 0)
+    (gr_text "4415.0000 mils" (at 113.6015 135.2226) (layer "Cmts.User")
+      (effects (font (size 1 1) (thickness 0.15)))
+    )
+    (format (units 3) (units_format 1) (precision 4))
+    (style (thickness 0.15) (arrow_length 1.27) (text_position_mode 0) (extension_height 0.58642) (extension_offset 0.5) keep_text_aligned)
+  )
+  (dimension (type orthogonal) (layer "Cmts.User")
+    (pts (xy 81.6356 36.6776) (xy 102.108 65.1256))
+    (height 86.614)
+    (orientation 0)
+    (gr_text "806.0000 mils" (at 91.8718 122.1416) (layer "Cmts.User")
+      (effects (font (size 1 1) (thickness 0.15)))
+    )
+    (format (units 3) (units_format 1) (precision 4))
+    (style (thickness 0.15) (arrow_length 1.27) (text_position_mode 0) (extension_height 0.58642) (extension_offset 0.5) keep_text_aligned)
+  )
+  (dimension (type orthogonal) (layer "Cmts.User")
+    (pts (xy 146.4564 65.1256) (xy 152.8834 102.0064))
+    (height 59.6392)
+    (orientation 0)
+    (gr_text "253.0315 mils" (at 149.6699 127) (layer "Cmts.User")
+      (effects (font (size 1 1) (thickness 0.15)))
+    )
+    (format (units 3) (units_format 1) (precision 4))
+    (style (thickness 0.15) (arrow_length 1.27) (text_position_mode 2) (extension_height 0.58642) (extension_offset 0.5) keep_text_aligned)
+  )
+  (dimension (type orthogonal) (layer "Cmts.User")
+    (pts (xy 102.108 65.1256) (xy 81.6856 36.6776))
+    (height -57.2008)
+    (orientation 1)
+    (gr_text "1120.0000 mils" (at 43.7572 50.9016 90) (layer "Cmts.User")
+      (effects (font (size 1 1) (thickness 0.15)))
+    )
+    (format (units 3) (units_format 1) (precision 4))
+    (style (thickness 0.15) (arrow_length 1.27) (text_position_mode 0) (extension_height 0.58642) (extension_offset 0.5) keep_text_aligned)
+  )
   (segment (start 93.599 88.582) (end 93.599 91.568) (width 0.25) (layer "F.Cu") (net 1))
